File: ethernet.kicad_sch (KiCad schematic)
At the start: 23 parts, among them IC7 LAN8651B1-E_LMX, J8 RJ45_LED, Y4 Crystal_GND24

Commit message: Add RJ45 connector from Wurth
Other:
- note added: "REFACTOR ALL, 10BASE-T1S is not good at all critical error"
Changed lines of the file:
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@@
+		)
+	)
+	(text "REFACTOR ALL, 10BASE-T1S is not good at all critical error"
+		(exclude_from_sim no)
+		(at 144.272 28.702 0)
+		(effects
+			(font
+				(size 1.27 1.27)
+			)
 		)
 	)
