File: usb-c.kicad_sch (KiCad schematic)
At the start: 14 parts, among them IC1 USBLC6-2SC6, IC2 632723100011, IC3 TCPP01-M12, Q1 STL11N3LLH6

Commit message: Homogenation of symbols
Parts:
- D1: renamed from D2; symbol weather-station-poc-sym:BAT54KFILM -> Device:D
- D2: renamed from D1; symbol weather-station-poc-sym:ESDA25P35-1U1M -> Device:D_Schottky
Changed lines of the file:
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@@
-	(wire
-		(pts
-			(xy 147.32 68.58) (xy 147.32 73.66)
-		)
-		(stroke
-			(width 0)
-			(type default)
-		)
-	)
 	(wire
 		(pts
@@
 	(wire
 		(pts
-			(xy 147.32 88.9) (xy 147.32 93.98)
+			(xy 147.32 83.82) (xy 147.32 93.98)
 		)
 		(stroke
@@
 	(wire
 		(pts
+			(xy 147.32 68.58) (xy 147.32 76.2)
+		)
+		(stroke
+			(width 0)
+			(type default)
+		)
+	)
+	(wire
+		(pts
 			(xy 180.34 81.28) (xy 190.5 81.28)
 		)
@@
 	(wire
 		(pts
+			(xy 147.32 106.68) (xy 156.21 106.68)
+		)
+		(stroke
+			(width 0)
+			(type default)
+		)
+	)
+	(wire
+		(pts
 			(xy 137.16 83.82) (xy 137.16 93.98)
 		)
@@
 	(wire
 		(pts
-			(xy 151.13 106.68) (xy 156.21 106.68)
-		)
-		(stroke
-			(width 0)
-			(type default)
-		)
-	)
-	(wire
-		(pts
 			(xy 157.48 68.58) (xy 157.48 71.12)
 		)
@@
 	(wire
 		(pts
-			(xy 130.81 106.68) (xy 135.89 106.68)
+			(xy 130.81 106.68) (xy 139.7 106.68)
 		)
 		(stroke
@@
 	)
 	(symbol
-		(lib_id "weather-station-poc-sym:ESDA25P35-1U1M")
-		(at 147.32 73.66 270)
+		(lib_id "Device:D_Schottky")
+		(at 147.32 80.01 270)
 		(unit 1)
 		(exclude_from_sim no)
@@
 		(on_board yes)
 		(dnp no)
-		(property "Reference" "D1"
-			(at 151.13 79.5019 90)
+		(property "Reference" "D2"
+			(at 150.114 77.978 90)
 			(effects
 				(font
@@
 		)
 		(property "Value" "ESDA25P35-1U1M"
-			(at 151.13 83.058 90)
+			(at 150.368 80.264 90)
 			(effects
 				(font
@@
 		)
 		(property "Footprint" "weather-station-poc-fp:ESDA25P351U1M"
-			(at 53.67 83.82 0)
+			(at 147.32 80.01 0)
+			(effects
+				(font
+					(size 1.27 1.27)
+				)
+				(hide yes)
+			)
+		)
+		(property "Datasheet" "~"
+			(at 147.32 80.01 0)
+			(effects
+				(font
+					(size 1.27 1.27)
+				)
+				(hide yes)
+			)
+		)
+		(property "Description" "Schottky diode"
+			(at 147.32 80.01 0)
+			(effects
+				(font
+					(size 1.27 1.27)
+				)
+				(hide yes)
+			)
+		)
+		(property "Height" "0.6"
+			(at -246.33 90.17 0)
 			(effects
 				(font
@@
 			)
 		)
-		(property "Datasheet" "https://www.st.com/resource/en/datasheet/esda20p50-1u1m.pdf"
-			(at -46.33 83.82 0)
+		(property "Mouser Part Number" "511-ESDA25P35-1U1M"
+			(at -346.33 90.17 0)
 			(effects
 				(font
@@
 			)
 		)
-		(property "Description" "STMicroelectronics ESDA25P35-1U1M, Uni-Directional TVS Diode, 1400W, 2-Pin QFN"
-			(at 147.32 73.66 0)
-			(effects
-				(font
-					(size 1.27 1.27)
-				)
-				(hide yes)
-			)
-		)
-		(property "Height" "0.6"
-			(at -246.33 83.82 0)
+		(property "Mouser Price/Stock" "https://www.mouser.co.uk/ProductDetail/STMicroelectronics/ESDA25P35-1U1M?qs=aVyJF2WnouQUWqgNP85ZrA%3D%3D"
+			(at -446.33 90.17 0)
 			(effects
 				(font
@@
 			)
 		)
-		(property "Mouser Part Number" "511-ESDA25P35-1U1M"
-			(at -346.33 83.82 0)
+		(property "Manufacturer_Name" "STMicroelectronics"
+			(at -546.33 90.17 0)
 			(effects
 				(font
@@
 			)
 		)
-		(property "Mouser Price/Stock" "https://www.mouser.co.uk/ProductDetail/STMicroelectronics/ESDA25P35-1U1M?qs=aVyJF2WnouQUWqgNP85ZrA%3D%3D"
-			(at -446.33 83.82 0)
-			(effects
-				(font
-					(size 1.27 1.27)
-				)
-				(justify left bottom)
-				(hide yes)
-			)
-		)
-		(property "Manufacturer_Name" "STMicroelectronics"
-			(at -546.33 83.82 0)
-			(effects
-				(font
-					(size 1.27 1.27)
-				)
-				(justify left bottom)
-				(hide yes)
-			)
-		)
 		(property "Manufacturer_Part_Number" "ESDA25P35-1U1M"
-			(at -646.33 83.82 0)
+			(at -646.33 90.17 0)
 			(effects
 				(font
@@
 			(project ""
 				(path "/38eb53bb-294e-46e4-ad59-fd355ca373b9/336d3e95-9b5f-4d37-8b5a-efff814cf96e"
-					(reference "D1")
+					(reference "D2")
 					(unit 1)
 				)
@@
 	)
 	(symbol
-		(lib_id "weather-station-poc-sym:BAT54KFILM")
-		(at 151.13 106.68 180)
+		(lib_id "Device:D")
+		(at 143.51 106.68 180)
 		(unit 1)
 		(exclude_from_sim no)
@@
 		(dnp no)
 		(fields_autoplaced yes)
-		(property "Reference" "D2"
-			(at 143.51 99.06 0)
+		(property "Reference" "D1"
+			(at 143.51 100.33 0)
 			(effects
 				(font
@@
 		)
 		(property "Value" "BAT54KFILM"
-			(at 143.51 101.6 0)
+			(at 143.51 102.87 0)
 			(effects
 				(font
@@
 		)
 		(property "Footprint" "weather-station-poc-fp:SODFL1608X70N"
-			(at 139.7 9.22 0)
-			(effects
-				(font
-					(size 1.27 1.27)
-				)
-				(justify left top)
-				(hide yes)
-			)
-		)
-		(property "Datasheet" "https://www.st.com/resource/en/datasheet/bat54.pdf"
-			(at 139.7 -90.78 0)
-			(effects
-				(font
-					(size 1.27 1.27)
-				)
-				(justify left top)
-				(hide yes)
-			)
-		)
-		(property "Description" "BAT54KFILM, Schottky Diode,  0.3A max, 40V 5ns, 2-Pin, SOD-523"
-			(at 151.13 106.68 0)
+			(at 143.51 106.68 0)
+			(effects
+				(font
+					(size 1.27 1.27)
+				)
+				(hide yes)
+			)
+		)
+		(property "Datasheet" "~"
+			(at 143.51 106.68 0)
+			(effects
+				(font
+					(size 1.27 1.27)
+				)
+				(hide yes)
+			)
+		)
+		(property "Description" "Diode"
+			(at 143.51 106.68 0)
 			(effects
 				(font
@@
 		)
 		(property "Height" "0.7"
-			(at 139.7 -290.78 0)
+			(at 132.08 -290.78 0)
 			(effects
 				(font
@@
 		)
 		(property "Mouser Part Number" "511-BAT54KFILM"
-			(at 139.7 -390.78 0)
+			(at 132.08 -390.78 0)
 			(effects
 				(font
@@
 		)
 		(property "Mouser Price/Stock" "https://www.mouser.co.uk/ProductDetail/STMicroelectronics/BAT54KFILM?qs=jZi1jxfVU95Y9ce6l3OT%252BA%3D%3D"
-			(at 139.7 -490.78 0)
+			(at 132.08 -490.78 0)
 			(effects
 				(font
@@
 		)
 		(property "Manufacturer_Name" "STMicroelectronics"
-			(at 139.7 -590.78 0)
+			(at 132.08 -590.78 0)
 			(effects
 				(font
@@
 		)
 		(property "Manufacturer_Part_Number" "BAT54KFILM"
-			(at 139.7 -690.78 0)
-			(effects
-				(font
-					(size 1.27 1.27)
-				)
-				(justify left top)
+			(at 132.08 -690.78 0)
+			(effects
+				(font
+					(size 1.27 1.27)
+				)
+				(justify left top)
+				(hide yes)
+			)
+		)
+		(property "Sim.Device" "D"
+			(at 143.51 106.68 0)
+			(effects
+				(font
+					(size 1.27 1.27)
+				)
+				(hide yes)
+			)
+		)
+		(property "Sim.Pins" "1=K 2=A"
+			(at 143.51 106.68 0)
+			(effects
+				(font
+					(size 1.27 1.27)
+				)
 				(hide yes)
 			)
@@
 			(project ""
 				(path "/38eb53bb-294e-46e4-ad59-fd355ca373b9/336d3e95-9b5f-4d37-8b5a-efff814cf96e"
-					(reference "D2")
+					(reference "D1")
 					(unit 1)
 				)

Commit message: Fill the cartridge for all schematics
Other:
- company: (none) -> Julien Cruvieux
- title: (none) -> USB C
Changed lines of the file:
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@@
 	(paper "A4")
 	(title_block
-		(date "2025-11-01")
+		(title "USB C")
+		(date "2025-12-26")
+		(rev "A")
+		(company "Julien Cruvieux")
 	)
 	(rectangle
