File: SecureElement.kicad_sch (KiCad schematic)
At the start: 3 parts, among them IC8 STSAFA110S8OCD03

Commit message: Reorganise synoptic schematic for better reading Closes #26
Parts:
- IC8: footprint SOIC127P600X175-8N -> weather-station-poc-fp:SOIC127P600X175-8N
Connections:
- net 3V3_STSAFEA110 renamed 3V3_STSAFE
- net SCL_STSAFEA110 renamed SCL_STSAFE
- net SDA_STSAFEA110 renamed SDA_STSAFE
- net ~{RESET}_STSAFEA110 renamed ~{RESET}_STSAFE
Other:
- note added: "STSAFE-A110"
- note added: "Secure element (STSAFE)"
Changed lines of the file:
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@@
 	(generator_version "9.0")
 	(paper "A4")
+	(rectangle
+		(start 100.33 80.01)
+		(end 179.07 106.68)
+		(stroke
+			(width 0)
+			(type dash)
+		)
+		(fill
+			(type none)
+		)
+	)
+	(text "STSAFE-A110"
+		(exclude_from_sim no)
+		(at 105.156 78.486 0)
+		(effects
+			(font
+				(size 1.27 1.27)
+			)
+		)
+	)
+	(text "Secure element (STSAFE)"
+		(exclude_from_sim no)
+		(at 140.716 23.368 0)
+		(effects
+			(font
+				(size 10 10)
+			)
+		)
+	)
 	(junction
 		(at 125.73 91.44)
@@
 		)
 	)
-	(hierarchical_label "3V3_STSAFEA110"
+	(hierarchical_label "3V3_STSAFE"
 		(shape input)
 		(at 111.76 91.44 180)
@@
 		)
 	)
-	(hierarchical_label "SCL_STSAFEA110"
+	(hierarchical_label "SCL_STSAFE"
 		(shape input)
 		(at 166.37 92.71 0)
@@
 		)
 	)
-	(hierarchical_label "~{RESET}_STSAFEA110"
+	(hierarchical_label "~{RESET}_STSAFE"
 		(shape input)
 		(at 134.62 88.9 180)
@@
 		)
 	)
-	(hierarchical_label "SDA_STSAFEA110"
+	(hierarchical_label "SDA_STSAFE"
 		(shape bidirectional)
 		(at 166.37 97.79 0)
@@
 			)
 		)
-		(property "Footprint" "SOIC127P600X175-8N"
+		(property "Footprint" "weather-station-poc-fp:SOIC127P600X175-8N"
 			(at 162.56 185.09 0)
 			(effects

Commit message: Continue schematic review
Changed lines of the file:
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@@
 	(text "STSAFE-A110"
 		(exclude_from_sim no)
-		(at 105.156 78.486 0)
+		(at 105.41 78.74 0)
 		(effects
 			(font
@@
 	(text "Secure element (STSAFE)"
 		(exclude_from_sim no)
-		(at 140.716 23.368 0)
+		(at 140.97 22.86 0)
 		(effects
 			(font

Commit message: Fix some little warnings and refomat schematics files
Parts:
- renumbered C92 to C94, C91 to C95
Changed lines of the file:
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@@
 		(dnp no)
 		(fields_autoplaced yes)
-		(property "Reference" "#PWR0140"
+		(property "Reference" "#PWR0155"
 			(at 125.73 105.41 0)
 			(effects
@@
 			(project ""
 				(path "/38eb53bb-294e-46e4-ad59-fd355ca373b9/9a031817-cce8-41f5-9861-f61338edb684"
-					(reference "#PWR0140")
+					(reference "#PWR0155")
 					(unit 1)
 				)
@@
 		(dnp no)
 		(fields_autoplaced yes)
-		(property "Reference" "C92"
+		(property "Reference" "C94"
 			(at 119.38 93.0909 0)
 			(effects
@@
 			(project ""
 				(path "/38eb53bb-294e-46e4-ad59-fd355ca373b9/9a031817-cce8-41f5-9861-f61338edb684"
-					(reference "C92")
+					(reference "C94")
 					(unit 1)
 				)
@@
 		(dnp no)
 		(fields_autoplaced yes)
-		(property "Reference" "C91"
+		(property "Reference" "C95"
 			(at 129.54 93.9799 0)
 			(effects
@@
 			(project "weather-station-poc"
 				(path "/38eb53bb-294e-46e4-ad59-fd355ca373b9/9a031817-cce8-41f5-9861-f61338edb684"
-					(reference "C91")
+					(reference "C95")
 					(unit 1)
 				)

Commit message: Reorder components number
Parts:
- renumbered C94 to C76, C95 to C77, IC8 to IC7
Changed lines of the file:
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@@
 		(dnp no)
 		(fields_autoplaced yes)
-		(property "Reference" "#PWR0155"
+		(property "Reference" "#PWR0121"
 			(at 125.73 105.41 0)
 			(effects
@@
 			(project ""
 				(path "/38eb53bb-294e-46e4-ad59-fd355ca373b9/9a031817-cce8-41f5-9861-f61338edb684"
-					(reference "#PWR0155")
+					(reference "#PWR0121")
 					(unit 1)
 				)
@@
 		(dnp no)
 		(fields_autoplaced yes)
-		(property "Reference" "IC8"
+		(property "Reference" "IC7"
 			(at 151.13 82.55 0)
 			(effects
@@
 			(project ""
 				(path "/38eb53bb-294e-46e4-ad59-fd355ca373b9/9a031817-cce8-41f5-9861-f61338edb684"
-					(reference "IC8")
+					(reference "IC7")
 					(unit 1)
 				)
@@
 		(dnp no)
 		(fields_autoplaced yes)
-		(property "Reference" "C94"
+		(property "Reference" "C76"
 			(at 119.38 93.0909 0)
 			(effects
@@
 			(project ""
 				(path "/38eb53bb-294e-46e4-ad59-fd355ca373b9/9a031817-cce8-41f5-9861-f61338edb684"
-					(reference "C94")
+					(reference "C76")
 					(unit 1)
 				)
@@
 		(dnp no)
 		(fields_autoplaced yes)
-		(property "Reference" "C95"
+		(property "Reference" "C77"
 			(at 129.54 93.9799 0)
 			(effects
@@
 			(project "weather-station-poc"
 				(path "/38eb53bb-294e-46e4-ad59-fd355ca373b9/9a031817-cce8-41f5-9861-f61338edb684"
-					(reference "C95")
+					(reference "C77")
 					(unit 1)
 				)

Commit message: Assign 0603 footprint to all capacitors
Parts:
- C77: footprint (none) -> Capacitor_SMD:C_0603_1608Metric_Pad1.08x0.95mm_HandSolder
Changed lines of the file:
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@@
 			)
 		)
-		(property "Footprint" ""
+		(property "Footprint" "Capacitor_SMD:C_0603_1608Metric_Pad1.08x0.95mm_HandSolder"
 			(at 126.6952 99.06 0)
 			(effects

Commit message: Assign 0603 footprints to all resistors
Parts:
- C76: footprint (none) -> Capacitor_SMD:CP_Elec_3x5.3
Changed lines of the file:
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@@
 			)
 		)
-		(property "Footprint" ""
+		(property "Footprint" "Capacitor_SMD:CP_Elec_3x5.3"
 			(at 116.5352 99.06 0)
 			(effects

Commit message: Fill the cartridge for all schematics
Other:
- company: (none) -> Julien Cruvieux
- title: (none) -> Secure elements
Changed lines of the file:
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@@
 	(generator_version "9.0")
 	(paper "A4")
+	(title_block
+		(title "Secure elements")
+		(date "2025-12-26")
+		(rev "A")
+		(company "Julien Cruvieux")
+	)
 	(rectangle
 		(start 100.33 80.01)

Commit message: Place MCU and its components around
Parts:
- renumbered C76 to C75, C77 to C76
Changed lines of the file:
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@@
 		(dnp no)
 		(fields_autoplaced yes)
-		(property "Reference" "#PWR0121"
+		(property "Reference" "#PWR0120"
 			(at 125.73 105.41 0)
 			(effects
@@
 			(project ""
 				(path "/38eb53bb-294e-46e4-ad59-fd355ca373b9/9a031817-cce8-41f5-9861-f61338edb684"
-					(reference "#PWR0121")
+					(reference "#PWR0120")
 					(unit 1)
 				)
@@
 		(dnp no)
 		(fields_autoplaced yes)
-		(property "Reference" "C76"
+		(property "Reference" "C75"
 			(at 119.38 93.0909 0)
 			(effects
@@
 			(project ""
 				(path "/38eb53bb-294e-46e4-ad59-fd355ca373b9/9a031817-cce8-41f5-9861-f61338edb684"
-					(reference "C76")
+					(reference "C75")
 					(unit 1)
 				)
@@
 		(dnp no)
 		(fields_autoplaced yes)
-		(property "Reference" "C77"
+		(property "Reference" "C76"
 			(at 129.54 93.9799 0)
 			(effects
@@
 			(project "weather-station-poc"
 				(path "/38eb53bb-294e-46e4-ad59-fd355ca373b9/9a031817-cce8-41f5-9861-f61338edb684"
-					(reference "C77")
+					(reference "C76")
 					(unit 1)
 				)
