File: SecureElement.kicad_sch (KiCad schematic)
At the start: 3 parts, among them IC7 STSAFA110S8OCD03

Commit message: Simplify S2LP schematic based on datasheet
Parts:
- renumbered C75 to C73, C76 to C74
Changed lines of the file:
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@@
 		(dnp no)
 		(fields_autoplaced yes)
-		(property "Reference" "#PWR0120"
+		(property "Reference" "#PWR0118"
 			(at 125.73 105.41 0)
 			(effects
@@
 			(project ""
 				(path "/38eb53bb-294e-46e4-ad59-fd355ca373b9/9a031817-cce8-41f5-9861-f61338edb684"
-					(reference "#PWR0120")
+					(reference "#PWR0118")
 					(unit 1)
 				)
@@
 		(dnp no)
 		(fields_autoplaced yes)
-		(property "Reference" "C75"
+		(property "Reference" "C73"
 			(at 119.38 93.0909 0)
 			(effects
@@
 			(project ""
 				(path "/38eb53bb-294e-46e4-ad59-fd355ca373b9/9a031817-cce8-41f5-9861-f61338edb684"
-					(reference "C75")
+					(reference "C73")
 					(unit 1)
 				)
@@
 		(dnp no)
 		(fields_autoplaced yes)
-		(property "Reference" "C76"
+		(property "Reference" "C74"
 			(at 129.54 93.9799 0)
 			(effects
@@
 			(project "weather-station-poc"
 				(path "/38eb53bb-294e-46e4-ad59-fd355ca373b9/9a031817-cce8-41f5-9861-f61338edb684"
-					(reference "C76")
+					(reference "C74")
 					(unit 1)
 				)

Commit message: Place all components on the PCB correctly
Parts:
- renumbered C73 to C74, C74 to C75
Changed lines of the file:
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@@
 		(dnp no)
 		(fields_autoplaced yes)
-		(property "Reference" "#PWR0118"
+		(property "Reference" "#PWR0119"
 			(at 125.73 105.41 0)
 			(effects
@@
 			(project ""
 				(path "/38eb53bb-294e-46e4-ad59-fd355ca373b9/9a031817-cce8-41f5-9861-f61338edb684"
-					(reference "#PWR0118")
+					(reference "#PWR0119")
 					(unit 1)
 				)
@@
 		(dnp no)
 		(fields_autoplaced yes)
-		(property "Reference" "C73"
+		(property "Reference" "C74"
 			(at 119.38 93.0909 0)
 			(effects
@@
 			(project ""
 				(path "/38eb53bb-294e-46e4-ad59-fd355ca373b9/9a031817-cce8-41f5-9861-f61338edb684"
-					(reference "C73")
+					(reference "C74")
 					(unit 1)
 				)
@@
 		(dnp no)
 		(fields_autoplaced yes)
-		(property "Reference" "C74"
+		(property "Reference" "C75"
 			(at 129.54 93.9799 0)
 			(effects
@@
 			(project "weather-station-poc"
 				(path "/38eb53bb-294e-46e4-ad59-fd355ca373b9/9a031817-cce8-41f5-9861-f61338edb684"
-					(reference "C74")
+					(reference "C75")
 					(unit 1)
 				)

Commit message: Prepare PCB for routing
Parts:
- removed C74: 10u, Capacitor_SMD:CP_Elec_3x5.3, symbol Device:C_Polarized
- added C74: 10u, Capacitor_SMD:C_0603_1608Metric_Pad1.08x0.95mm_HandSolder, symbol Device:C
Connections:
- net 3V3_STSAFE: now also C74.1
- net GND: now also C74.2
Changed lines of the file:
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@@
+	(wire
+		(pts
+			(xy 111.76 91.44) (xy 115.57 91.44)
+		)
+		(stroke
+			(width 0)
+			(type default)
+		)
+	)
+	(wire
+		(pts
+			(xy 125.73 99.06) (xy 135.89 99.06)
+		)
+		(stroke
+			(width 0)
+			(type default)
+		)
+	)
+	(wire
+		(pts
+			(xy 134.62 88.9) (xy 135.89 88.9)
+		)
+		(stroke
+			(width 0)
+			(type default)
+		)
+	)
+	(wire
+		(pts
+			(xy 135.89 97.79) (xy 135.89 99.06)
+		)
+		(stroke
+			(width 0)
+			(type default)
+		)
+	)
+	(wire
+		(pts
+			(xy 135.89 88.9) (xy 135.89 90.17)
+		)
+		(stroke
+			(width 0)
+			(type default)
+		)
+	)
 	(wire
 		(pts
 			(xy 115.57 91.44) (xy 125.73 91.44)
-		)
-		(stroke
-			(width 0)
-			(type default)
-		)
-	)
-	(wire
-		(pts
-			(xy 111.76 91.44) (xy 115.57 91.44)
-		)
-		(stroke
-			(width 0)
-			(type default)
-		)
-	)
-	(wire
-		(pts
-			(xy 125.73 99.06) (xy 135.89 99.06)
-		)
-		(stroke
-			(width 0)
-			(type default)
-		)
-	)
-	(wire
-		(pts
-			(xy 134.62 88.9) (xy 135.89 88.9)
-		)
-		(stroke
-			(width 0)
-			(type default)
-		)
-	)
-	(wire
-		(pts
-			(xy 135.89 97.79) (xy 135.89 99.06)
-		)
-		(stroke
-			(width 0)
-			(type default)
-		)
-	)
-	(wire
-		(pts
-			(xy 135.89 88.9) (xy 135.89 90.17)
 		)
 		(stroke
@@
 	)
 	(symbol
+		(lib_id "Device:C")
+		(at 115.57 95.25 0)
+		(unit 1)
+		(exclude_from_sim no)
+		(in_bom yes)
+		(on_board yes)
+		(dnp no)
+		(fields_autoplaced yes)
+		(property "Reference" "C74"
+			(at 119.38 93.9799 0)
+			(effects
+				(font
+					(size 1.27 1.27)
+				)
+				(justify left)
+			)
+		)
+		(property "Value" "10u"
+			(at 119.38 96.5199 0)
+			(effects
+				(font
+					(size 1.27 1.27)
+				)
+				(justify left)
+			)
+		)
+		(property "Footprint" "Capacitor_SMD:C_0603_1608Metric_Pad1.08x0.95mm_HandSolder"
+			(at 116.5352 99.06 0)
+			(effects
+				(font
+					(size 1.27 1.27)
+				)
+				(hide yes)
+			)
+		)
+		(property "Datasheet" "~"
+			(at 115.57 95.25 0)
+			(effects
+				(font
+					(size 1.27 1.27)
+				)
+				(hide yes)
+			)
+		)
+		(property "Description" "Unpolarized capacitor"
+			(at 115.57 95.25 0)
+			(effects
+				(font
+					(size 1.27 1.27)
+				)
+				(hide yes)
+			)
+		)
+		(pin "2"
+		)
+		(pin "1"
+		)
+		(instances
+			(project "weather-station-poc"
+				(path "/38eb53bb-294e-46e4-ad59-fd355ca373b9/9a031817-cce8-41f5-9861-f61338edb684"
+					(reference "C74")
+					(unit 1)
+				)
+			)
+		)
+	)
+	(symbol
 		(lib_id "weather-station-poc-sym:STSAFA110S8OCD03")
 		(at 135.89 90.17 0)
@@
 					(unit 1)
 				)
-			)
-		)
-	)
-	(symbol
-		(lib_id "Device:C_Polarized")
-		(at 115.57 95.25 0)
-		(unit 1)
-		(exclude_from_sim no)
-		(in_bom yes)
-		(on_board yes)
-		(dnp no)
-		(fields_autoplaced yes)
-		(property "Reference" "C74"
-			(at 119.38 93.0909 0)
-			(effects
-				(font
-					(size 1.27 1.27)
-				)
-				(justify left)
-			)
-		)
-		(property "Value" "10u"
-			(at 119.38 95.6309 0)
-			(effects
-				(font
-					(size 1.27 1.27)
-				)
-				(justify left)
-			)
-		)
-		(property "Footprint" "Capacitor_SMD:CP_Elec_3x5.3"
-			(at 116.5352 99.06 0)
-			(effects
-				(font
-					(size 1.27 1.27)
-				)
-				(hide yes)
-			)
-		)
-		(property "Datasheet" "~"
-			(at 115.57 95.25 0)
-			(effects
-				(font
-					(size 1.27 1.27)
-				)
-				(hide yes)
-			)
-		)
-		(property "Description" "Polarized capacitor"
-			(at 115.57 95.25 0)
-			(effects
-				(font
-					(size 1.27 1.27)
-				)
-				(hide yes)
-			)
-		)
-		(pin "1"
-		)
-		(pin "2"
-		)
-		(instances
-			(project ""
-				(path "/38eb53bb-294e-46e4-ad59-fd355ca373b9/9a031817-cce8-41f5-9861-f61338edb684"
-					(reference "C74")
-					(unit 1)
-				)

Commit message: Update schematic to Kicad 10
Changed lines of the file:
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@@
 (kicad_sch
-	(version 20250114)
+	(version 20260306)
 	(generator "eeschema")
-	(generator_version "9.0")
+	(generator_version "10.0")
 	(paper "A4")
 	(title_block
@@
 	)
 	(rectangle
-		(start 100.33 80.01)
-		(end 179.07 106.68)
+		(start 97.79 80.01)
+		(end 180.34 106.68)
 		(stroke
 			(width 0)
@@
 	(text "STSAFE-A110"
 		(exclude_from_sim no)
-		(at 105.41 78.74 0)
+		(at 104.14 78.74 0)
 		(effects
 			(font
@@
 		(at 125.73 99.06 0)
 		(unit 1)
+		(body_style 1)
 		(exclude_from_sim no)
 		(in_bom yes)
 		(on_board yes)
+		(in_pos_files yes)
 		(dnp no)
 		(fields_autoplaced yes)
 		(property "Reference" "#PWR0119"
 			(at 125.73 105.41 0)
-			(effects
-				(font
-					(size 1.27 1.27)
-				)
-				(hide yes)
+			(hide yes)
+			(show_name no)
+			(do_not_autoplace no)
+			(effects
+				(font
+					(size 1.27 1.27)
+				)
 			)
 		)
 		(property "Value" "GND"
 			(at 125.73 104.14 0)
+			(show_name no)
+			(do_not_autoplace no)
 			(effects
 				(font
@@
 		(property "Footprint" ""
 			(at 125.73 99.06 0)
-			(effects
-				(font
-					(size 1.27 1.27)
-				)
-				(hide yes)
+			(hide yes)
+			(show_name no)
+			(do_not_autoplace no)
+			(effects
+				(font
+					(size 1.27 1.27)
+				)
 			)
 		)
 		(property "Datasheet" ""
 			(at 125.73 99.06 0)
-			(effects
-				(font
-					(size 1.27 1.27)
-				)
-				(hide yes)
+			(hide yes)
+			(show_name no)
+			(do_not_autoplace no)
+			(effects
+				(font
+					(size 1.27 1.27)
+				)
 			)
 		)
 		(property "Description" "Power symbol creates a global label with name \"GND\" , ground"
 			(at 125.73 99.06 0)
-			(effects
-				(font
-					(size 1.27 1.27)
-				)
-				(hide yes)
+			(hide yes)
+			(show_name no)
+			(do_not_autoplace no)
+			(effects
+				(font
+					(size 1.27 1.27)
+				)
 			)
 		)
@@
 		)
 		(instances
-			(project ""
+			(project "weather-station-poc"
 				(path "/38eb53bb-294e-46e4-ad59-fd355ca373b9/9a031817-cce8-41f5-9861-f61338edb684"
 					(reference "#PWR0119")
@@
 		(at 115.57 95.25 0)
 		(unit 1)
+		(body_style 1)
 		(exclude_from_sim no)
 		(in_bom yes)
 		(on_board yes)
+		(in_pos_files yes)
 		(dnp no)
 		(fields_autoplaced yes)
 		(property "Reference" "C74"
 			(at 119.38 93.9799 0)
+			(show_name no)
+			(do_not_autoplace no)
 			(effects
 				(font
@@
 		(property "Value" "10u"
 			(at 119.38 96.5199 0)
+			(show_name no)
+			(do_not_autoplace no)
 			(effects
 				(font
@@
 		(property "Footprint" "Capacitor_SMD:C_0603_1608Metric_Pad1.08x0.95mm_HandSolder"
 			(at 116.5352 99.06 0)
-			(effects
-				(font
-					(size 1.27 1.27)
-				)
-				(hide yes)
-			)
-		)
-		(property "Datasheet" "~"
+			(hide yes)
+			(show_name no)
+			(do_not_autoplace no)
+			(effects
+				(font
+					(size 1.27 1.27)
+				)
+			)
+		)
+		(property "Datasheet" ""
 			(at 115.57 95.25 0)
-			(effects
-				(font
-					(size 1.27 1.27)
-				)
-				(hide yes)
+			(hide yes)
+			(show_name no)
+			(do_not_autoplace no)
+			(effects
+				(font
+					(size 1.27 1.27)
+				)
 			)
 		)
 		(property "Description" "Unpolarized capacitor"
 			(at 115.57 95.25 0)
-			(effects
-				(font
-					(size 1.27 1.27)
-				)
-				(hide yes)
+			(hide yes)
+			(show_name no)
+			(do_not_autoplace no)
+			(effects
+				(font
+					(size 1.27 1.27)
+				)
 			)
 		)
@@
 		(at 135.89 90.17 0)
 		(unit 1)
+		(body_style 1)
 		(exclude_from_sim no)
 		(in_bom yes)
 		(on_board yes)
+		(in_pos_files yes)
 		(dnp no)
 		(fields_autoplaced yes)
 		(property "Reference" "IC7"
 			(at 151.13 82.55 0)
+			(show_name no)
+			(do_not_autoplace no)
 			(effects
 				(font
@@
 		(property "Value" "STSAFA110S8OCD03"
 			(at 151.13 85.09 0)
+			(show_name no)
+			(do_not_autoplace no)
 			(effects
 				(font
@@
 		(property "Footprint" "weather-station-poc-fp:SOIC127P600X175-8N"
 			(at 162.56 185.09 0)
-			(effects
-				(font
-					(size 1.27 1.27)
-				)
-				(justify left top)
-				(hide yes)
+			(hide yes)
+			(show_name no)
+			(do_not_autoplace no)
+			(effects
+				(font
+					(size 1.27 1.27)
+				)
+				(justify left top)
 			)
 		)
 		(property "Datasheet" "https://www.st.com/resource/en/datasheet/stsafe-a110.pdf"
 			(at 162.56 285.09 0)
-			(effects
-				(font
-					(size 1.27 1.27)
-				)
-				(justify left top)
-				(hide yes)
+			(hide yes)
+			(show_name no)
+			(do_not_autoplace no)
+			(effects
+				(font
+					(size 1.27 1.27)
+				)
+				(justify left top)
 			)
 		)
 		(property "Description" "Authentication, state-of-the-art security for peripherals and IoT devices"
 			(at 135.89 90.17 0)
-			(effects
-				(font
-					(size 1.27 1.27)
-				)
-				(hide yes)
+			(hide yes)
+			(show_name no)
+			(do_not_autoplace no)
+			(effects
+				(font
+					(size 1.27 1.27)
+				)
 			)
 		)
 		(property "Height" "1.75"
 			(at 162.56 485.09 0)
-			(effects
-				(font
-					(size 1.27 1.27)
-				)
-				(justify left top)
-				(hide yes)
+			(hide yes)
+			(show_name no)
+			(do_not_autoplace no)
+			(effects
+				(font
+					(size 1.27 1.27)
+				)
+				(justify left top)
 			)
 		)
 		(property "Mouser Part Number" "511-STSAFA110S8OCD03"
 			(at 162.56 585.09 0)
-			(effects
-				(font
-					(size 1.27 1.27)
-				)
-				(justify left top)
-				(hide yes)
+			(hide yes)
+			(show_name no)
+			(do_not_autoplace no)
+			(effects
+				(font
+					(size 1.27 1.27)
+				)
+				(justify left top)
 			)
 		)
 		(property "Mouser Price/Stock" "https://www.mouser.co.uk/ProductDetail/STMicroelectronics/STSAFA110S8OCD03?qs=7%2F6SraaimPRtuR%252B2wUZjKw%3D%3D"
 			(at 162.56 685.09 0)
-			(effects
-				(font
-					(size 1.27 1.27)
-				)
-				(justify left top)
-				(hide yes)
+			(hide yes)
+			(show_name no)
+			(do_not_autoplace no)
+			(effects
+				(font
+					(size 1.27 1.27)
+				)
+				(justify left top)
 			)
 		)
 		(property "Manufacturer_Name" "STMicroelectronics"
 			(at 162.56 785.09 0)
-			(effects
-				(font
-					(size 1.27 1.27)
-				)
-				(justify left top)
-				(hide yes)
+			(hide yes)
+			(show_name no)
+			(do_not_autoplace no)
+			(effects
+				(font
+					(size 1.27 1.27)
+				)
+				(justify left top)
 			)
 		)
 		(property "Manufacturer_Part_Number" "STSAFA110S8OCD03"
 			(at 162.56 885.09 0)
-			(effects
-				(font
-					(size 1.27 1.27)
-				)
-				(justify left top)
-				(hide yes)
+			(hide yes)
+			(show_name no)
+			(do_not_autoplace no)
+			(effects
+				(font
+					(size 1.27 1.27)
+				)
+				(justify left top)
 			)
 		)
@@
 		)
 		(instances
-			(project ""
+			(project "weather-station-poc"
 				(path "/38eb53bb-294e-46e4-ad59-fd355ca373b9/9a031817-cce8-41f5-9861-f61338edb684"
 					(reference "IC7")
@@
 		(at 125.73 95.25 0)
 		(unit 1)
+		(body_style 1)
 		(exclude_from_sim no)
 		(in_bom yes)
 		(on_board yes)
+		(in_pos_files yes)
 		(dnp no)
 		(fields_autoplaced yes)
 		(property "Reference" "C75"
 			(at 129.54 93.9799 0)
+			(show_name no)
+			(do_not_autoplace no)
 			(effects
 				(font
@@
 		(property "Value" "100n"
 			(at 129.54 96.5199 0)
+			(show_name no)
+			(do_not_autoplace no)
 			(effects
 				(font
@@
 		(property "Footprint" "Capacitor_SMD:C_0603_1608Metric_Pad1.08x0.95mm_HandSolder"
 			(at 126.6952 99.06 0)
-			(effects
-				(font
-					(size 1.27 1.27)
-				)
-				(hide yes)
-			)
-		)
-		(property "Datasheet" "~"
+			(hide yes)
+			(show_name no)
+			(do_not_autoplace no)
+			(effects
+				(font
+					(size 1.27 1.27)
+				)
+			)
+		)
+		(property "Datasheet" ""
 			(at 125.73 95.25 0)
-			(effects
-				(font
-					(size 1.27 1.27)
-				)
-				(hide yes)
+			(hide yes)
+			(show_name no)
+			(do_not_autoplace no)
+			(effects
+				(font
+					(size 1.27 1.27)
+				)
 			)
 		)
 		(property "Description" "Unpolarized capacitor"
 			(at 125.73 95.25 0)
-			(effects
-				(font
-					(size 1.27 1.27)
-				)
-				(hide yes)
-			)
-		)
+			(hide yes)
+			(show_name no)
+			(do_not_autoplace no)
+			(effects
+				(font
+					(size 1.27 1.27)
+				)
+			)
+		)

Commit message: Add tests points with 5015 footprint for practicity
Other:
- moved on the sheet: C74, C75, IC7
Changed lines of the file:
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@@
 	)
 	(rectangle
-		(start 97.79 80.01)
-		(end 180.34 106.68)
+		(start 104.14 81.28)
+		(end 186.69 107.95)
 		(stroke
 			(width 0)
@@
 	(text "STSAFE-A110"
 		(exclude_from_sim no)
-		(at 104.14 78.74 0)
+		(at 110.49 80.01 0)
 		(effects
 			(font
@@
 	)
 	(junction
-		(at 125.73 91.44)
+		(at 132.08 92.71)
 		(diameter 0)
 		(color 0 0 0 0)
 	)
 	(junction
-		(at 115.57 91.44)
+		(at 121.92 92.71)
 		(diameter 0)
 		(color 0 0 0 0)
 	)
 	(junction
-		(at 125.73 99.06)
+		(at 132.08 100.33)
 		(diameter 0)
 		(color 0 0 0 0)
 	)
 	(no_connect
-		(at 166.37 95.25)
+		(at 172.72 96.52)
 	)
 	(no_connect
-		(at 166.37 90.17)
+		(at 172.72 91.44)
 	)
 	(no_connect
-		(at 135.89 95.25)
-	)
-	(wire
-		(pts
-			(xy 111.76 91.44) (xy 115.57 91.44)
-		)
-		(stroke
-			(width 0)
-			(type default)
-		)
-	)
-	(wire
-		(pts
-			(xy 125.73 99.06) (xy 135.89 99.06)
-		)
-		(stroke
-			(width 0)
-			(type default)
-		)
-	)
-	(wire
-		(pts
-			(xy 134.62 88.9) (xy 135.89 88.9)
-		)
-		(stroke
-			(width 0)
-			(type default)
-		)
-	)
-	(wire
-		(pts
-			(xy 135.89 97.79) (xy 135.89 99.06)
-		)
-		(stroke
-			(width 0)
-			(type default)
-		)
-	)
-	(wire
-		(pts
-			(xy 135.89 88.9) (xy 135.89 90.17)
-		)
-		(stroke
-			(width 0)
-			(type default)
-		)
-	)
-	(wire
-		(pts
-			(xy 115.57 91.44) (xy 125.73 91.44)
-		)
-		(stroke
-			(width 0)
-			(type default)
-		)
-	)
-	(wire
-		(pts
-			(xy 125.73 91.44) (xy 135.89 91.44)
-		)
-		(stroke
-			(width 0)
-			(type default)
-		)
-	)
-	(wire
-		(pts
-			(xy 115.57 99.06) (xy 125.73 99.06)
-		)
-		(stroke
-			(width 0)
-			(type default)
-		)
-	)
-	(wire
-		(pts
-			(xy 135.89 92.71) (xy 135.89 91.44)
+		(at 142.24 96.52)
+	)
+	(wire
+		(pts
+			(xy 118.11 92.71) (xy 121.92 92.71)
+		)
+		(stroke
+			(width 0)
+			(type default)
+		)
+	)
+	(wire
+		(pts
+			(xy 132.08 100.33) (xy 142.24 100.33)
+		)
+		(stroke
+			(width 0)
+			(type default)
+		)
+	)
+	(wire
+		(pts
+			(xy 140.97 90.17) (xy 142.24 90.17)
+		)
+		(stroke
+			(width 0)
+			(type default)
+		)
+	)
+	(wire
+		(pts
+			(xy 142.24 99.06) (xy 142.24 100.33)
+		)
+		(stroke
+			(width 0)
+			(type default)
+		)
+	)
+	(wire
+		(pts
+			(xy 142.24 90.17) (xy 142.24 91.44)
+		)
+		(stroke
+			(width 0)
+			(type default)
+		)
+	)
+	(wire
+		(pts
+			(xy 121.92 92.71) (xy 132.08 92.71)
+		)
+		(stroke
+			(width 0)
+			(type default)
+		)
+	)
+	(wire
+		(pts
+			(xy 132.08 92.71) (xy 142.24 92.71)
+		)
+		(stroke
+			(width 0)
+			(type default)
+		)
+	)
+	(wire
+		(pts
+			(xy 121.92 100.33) (xy 132.08 100.33)
+		)
+		(stroke
+			(width 0)
+			(type default)
+		)
+	)
+	(wire
+		(pts
+			(xy 142.24 93.98) (xy 142.24 92.71)
 		)
 		(stroke
@@
 	(hierarchical_label "3V3_STSAFE"
 		(shape input)
-		(at 111.76 91.44 180)
+		(at 118.11 92.71 180)
 		(effects
 			(font
@@
 	(hierarchical_label "SCL_STSAFE"
 		(shape input)
-		(at 166.37 92.71 0)
+		(at 172.72 93.98 0)
 		(effects
 			(font
@@
 	(hierarchical_label "~{RESET}_STSAFE"
 		(shape input)
-		(at 134.62 88.9 180)
+		(at 140.97 90.17 180)
 		(effects
 			(font
@@
 	(hierarchical_label "SDA_STSAFE"
 		(shape bidirectional)
-		(at 166.37 97.79 0)
+		(at 172.72 99.06 0)
 		(effects
 			(font
@@
 	(symbol
 		(lib_id "power:GND")
-		(at 125.73 99.06 0)
+		(at 132.08 100.33 0)
 		(unit 1)
 		(body_style 1)
@@
 		(dnp no)
 		(fields_autoplaced yes)
-		(property "Reference" "#PWR0119"
-			(at 125.73 105.41 0)
+		(property "Reference" "#PWR0127"
+			(at 132.08 106.68 0)
 			(hide yes)
 			(show_name no)
@@
 		)
 		(property "Value" "GND"
-			(at 125.73 104.14 0)
+			(at 132.08 105.41 0)
 			(show_name no)
 			(do_not_autoplace no)
@@
 		)
 		(property "Footprint" ""
-			(at 125.73 99.06 0)
+			(at 132.08 100.33 0)
 			(hide yes)
 			(show_name no)
@@
 		)
 		(property "Datasheet" ""
-			(at 125.73 99.06 0)
+			(at 132.08 100.33 0)
 			(hide yes)
 			(show_name no)
@@
 		)
 		(property "Description" "Power symbol creates a global label with name \"GND\" , ground"
-			(at 125.73 99.06 0)
+			(at 132.08 100.33 0)
 			(hide yes)
 			(show_name no)
@@
 			(project "weather-station-poc"
 				(path "/38eb53bb-294e-46e4-ad59-fd355ca373b9/9a031817-cce8-41f5-9861-f61338edb684"
-					(reference "#PWR0119")
+					(reference "#PWR0127")
 					(unit 1)
 				)
@@
 	(symbol
 		(lib_id "Device:C")
-		(at 115.57 95.25 0)
+		(at 121.92 96.52 0)
 		(unit 1)
 		(body_style 1)
@@
 		(fields_autoplaced yes)
 		(property "Reference" "C74"
-			(at 119.38 93.9799 0)
+			(at 125.73 95.2499 0)
 			(show_name no)
 			(do_not_autoplace no)
@@
 		)
 		(property "Value" "10u"
-			(at 119.38 96.5199 0)
+			(at 125.73 97.7899 0)
 			(show_name no)
 			(do_not_autoplace no)
@@
 		)
 		(property "Footprint" "Capacitor_SMD:C_0603_1608Metric_Pad1.08x0.95mm_HandSolder"
-			(at 116.5352 99.06 0)
+			(at 122.8852 100.33 0)
 			(hide yes)
 			(show_name no)
@@
 		)
 		(property "Datasheet" ""
-			(at 115.57 95.25 0)
+			(at 121.92 96.52 0)
 			(hide yes)
 			(show_name no)
@@
 		)
 		(property "Description" "Unpolarized capacitor"
-			(at 115.57 95.25 0)
+			(at 121.92 96.52 0)
 			(hide yes)
 			(show_name no)
@@
 	(symbol
 		(lib_id "weather-station-poc-sym:STSAFA110S8OCD03")
-		(at 135.89 90.17 0)
+		(at 142.24 91.44 0)
 		(unit 1)
 		(body_style 1)
@@
 		(fields_autoplaced yes)
 		(property "Reference" "IC7"
-			(at 151.13 82.55 0)
+			(at 157.48 83.82 0)
 			(show_name no)
 			(do_not_autoplace no)
@@
 		)
 		(property "Value" "STSAFA110S8OCD03"
-			(at 151.13 85.09 0)
+			(at 157.48 86.36 0)
 			(show_name no)
 			(do_not_autoplace no)
@@
 		)
 		(property "Footprint" "weather-station-poc-fp:SOIC127P600X175-8N"
-			(at 162.56 185.09 0)
+			(at 168.91 186.36 0)
 			(hide yes)
 			(show_name no)
@@
 		)
 		(property "Datasheet" "https://www.st.com/resource/en/datasheet/stsafe-a110.pdf"
-			(at 162.56 285.09 0)
+			(at 168.91 286.36 0)
 			(hide yes)
 			(show_name no)
@@
 		)
 		(property "Description" "Authentication, state-of-the-art security for peripherals and IoT devices"
-			(at 135.89 90.17 0)
+			(at 142.24 91.44 0)
 			(hide yes)
 			(show_name no)
@@
 		)
 		(property "Height" "1.75"
-			(at 162.56 485.09 0)
+			(at 168.91 486.36 0)
 			(hide yes)
 			(show_name no)
@@
 		)
 		(property "Mouser Part Number" "511-STSAFA110S8OCD03"
-			(at 162.56 585.09 0)
+			(at 168.91 586.36 0)
 			(hide yes)
 			(show_name no)
@@
 		)
 		(property "Mouser Price/Stock" "https://www.mouser.co.uk/ProductDetail/STMicroelectronics/STSAFA110S8OCD03?qs=7%2F6SraaimPRtuR%252B2wUZjKw%3D%3D"
-			(at 162.56 685.09 0)
+			(at 168.91 686.36 0)
 			(hide yes)
 			(show_name no)
@@
 		)
 		(property "Manufacturer_Name" "STMicroelectronics"
-			(at 162.56 785.09 0)
+			(at 168.91 786.36 0)
 			(hide yes)
 			(show_name no)
@@
 		)
 		(property "Manufacturer_Part_Number" "STSAFA110S8OCD03"
-			(at 162.56 885.09 0)
+			(at 168.91 886.36 0)
 			(hide yes)
 			(show_name no)
@@
 	(symbol
 		(lib_id "Device:C")
-		(at 125.73 95.25 0)
+		(at 132.08 96.52 0)
 		(unit 1)
 		(body_style 1)
@@
 		(fields_autoplaced yes)
 		(property "Reference" "C75"
-			(at 129.54 93.9799 0)
+			(at 135.89 95.2499 0)
 			(show_name no)
 			(do_not_autoplace no)
@@
 		)
 		(property "Value" "100n"
-			(at 129.54 96.5199 0)
+			(at 135.89 97.7899 0)
 			(show_name no)
 			(do_not_autoplace no)
@@
 		)
 		(property "Footprint" "Capacitor_SMD:C_0603_1608Metric_Pad1.08x0.95mm_HandSolder"
-			(at 126.6952 99.06 0)
+			(at 133.0452 100.33 0)
 			(hide yes)
 			(show_name no)
@@
 		)
 		(property "Datasheet" ""
-			(at 125.73 95.25 0)
+			(at 132.08 96.52 0)
 			(hide yes)
 			(show_name no)
@@
 		)
 		(property "Description" "Unpolarized capacitor"
-			(at 125.73 95.25 0)
-			(hide yes)
-			(show_name no)
+			(at 132.08 96.52 0)
+			(hide yes)
+			(show_name no)
