File: SecureElement.kicad_sch (KiCad schematic)
At the start: 3 parts, among them IC7 STSAFA110S8OCD03

Commit message: Complete all references for components
Modifgy Y1 and Y2 capacitors footprint from 0603 to 0402
Modify footprint of SWD connector
Parts:
- C74: Manufacturer_Name (none) -> Murata Electronics; Manufacturer_Part_Number (none) -> GRM188Z71A106KA73D
- C75: Manufacturer_Name (none) -> Wurth Elektronik; Manufacturer_Part_Number (none) -> 885012206020
Changed lines of the file:
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@@
 			)
 		)
-		(property "Datasheet" ""
+		(property "Datasheet" "https://eu.mouser.com/datasheet/3/76/2/GRM188Z71A106KA73_01A.pdf"
 			(at 121.92 96.52 0)
 			(hide yes)
@@
 		)
 		(property "Description" "Unpolarized capacitor"
+			(at 121.92 96.52 0)
+			(hide yes)
+			(show_name no)
+			(do_not_autoplace no)
+			(effects
+				(font
+					(size 1.27 1.27)
+				)
+			)
+		)
+		(property "Manufacturer_Name" "Murata Electronics"
+			(at 121.92 96.52 0)
+			(hide yes)
+			(show_name no)
+			(do_not_autoplace no)
+			(effects
+				(font
+					(size 1.27 1.27)
+				)
+			)
+		)
+		(property "Manufacturer_Part_Number" "GRM188Z71A106KA73D"
 			(at 121.92 96.52 0)
 			(hide yes)
@@
 			)
 		)
-		(property "Datasheet" ""
+		(property "Datasheet" "https://www.we-online.com/components/products/datasheet/885012206020.pdf"
 			(at 132.08 96.52 0)
 			(hide yes)
@@
 			(at 132.08 96.52 0)
 			(hide yes)
+			(show_name no)
+			(do_not_autoplace no)
+			(effects
+				(font
+					(size 1.27 1.27)
+				)
+			)
+		)
+		(property "Manufacturer_Name" "Wurth Elektronik"
+			(at 132.08 96.52 0)
+			(hide yes)
+			(show_name no)
+			(do_not_autoplace no)
+			(effects
+				(font
+					(size 1.27 1.27)
+				)
+			)
+		)
+		(property "Manufacturer_Part_Number" "885012206020"
+			(at 132.08 96.52 0)
+			(hide yes)
