File: block-diagram.kicad_sch (KiCad schematic)
At the start: 0 parts

Commit message: Fill the cartridge for all schematics
Other:
- company: (none) -> Julien Cruvieux
- title: (none) -> Block diagram
Changed lines of the file:
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@@
 	(generator_version "9.0")
 	(paper "A4")
+	(title_block
+		(title "Block diagram")
+		(date "2025-12-26")
+		(rev "A")
+		(company "Julien Cruvieux")
+	)
 	(image
 		(at 92.9409 157.2439)
