File: block-diagram.kicad_sch (KiCad schematic)
At the start: 0 parts

Commit message: Set I2C address for BMP sensors and document address
Other:
- note added: "7628 FR DK = 4.4 So 0.3mm trace width => 54.9 ohms For USB differentials pairs, 0.3mm trace width and 0.3mm spacing => 96.4 ohms (90 ohms +/- 10% for USB) Calculation according PCB way impedance calculator : (https://www.pcbway.com/pcb_prototype/impedance_calculator.html)"
- note added: "JLCPCB stackup"
- note added: "L1 and L4 have a direct return paths through solid ground plane on L2 and L3. But Pwr on L1 is perhaps an issue in terms of EMC ?"
- note added: "PCB build up"
