File: lcd.kicad_sch (KiCad schematic)
At the start: 2 parts, among them J6 687140149022, J7 687110183622

Commit message: Move SWD debug connector from debug sheet to MCU sheet
Other:
- moved on the sheet: J6, J7

Commit message: Rename backlight power pins
Connections:
- net VLED+_LCD renamed +VBacklight_LCD
- net VLED-_LCD renamed -VBacklight_LCD
Changed lines of the file:
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@@
 		)
 	)
-	(hierarchical_label "VLED+_LCD"
+	(hierarchical_label "+VBacklight_LCD"
 		(shape input)
 		(at 118.11 54.61 0)
@@
 		)
 	)
-	(hierarchical_label "VLED-_LCD"
+	(hierarchical_label "-VBacklight_LCD"
 		(shape output)
 		(at 118.11 52.07 0)

Commit message: Add RVT50HQTFWCA0 documentation link into a connector properpty
Parts:
- J6, J7: LCD documentation (none) -> https://download.riverdi.com/RVT50HQTFWCA0/DS_RVT50HQTFWCA0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
Other:
- note added: "RVT50HQTFWCA0 LCD screen"
- note removed: "TFT LCD screen"
Changed lines of the file:
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@@
 		)
 	)
-	(text "TFT LCD screen"
+	(text "RVT50HQTFWCA0 LCD screen"
 		(exclude_from_sim no)
 		(at 149.86 24.13 0)
@@
 			)
 		)
+		(property "LCD documentation" "https://download.riverdi.com/RVT50HQTFWCA0/DS_RVT50HQTFWCA0%20V2.0A_Rev.1.1.pdf?_gl=1*nkotui*_gcl_au*MTM1MDU3OTk5Ny4xNzg2NDU0Mzc2Li0uLS4xNzg2NDU0MzgxLjE5ODgzMTQ2NTEuMTc4NjQ1NDM4MS4xNzg2NDU0Mzgx"
+			(at 92.71 52.07 0)
+			(hide yes)
+			(show_name no)
+			(do_not_autoplace no)
+			(effects
+				(font
+					(size 1.27 1.27)
+				)
+			)
+		)
 		(pin "3"
 		)
@@
 			)
 		)
+		(property "LCD documentation" "https://download.riverdi.com/RVT50HQTFWCA0/DS_RVT50HQTFWCA0%20V2.0A_Rev.1.1.pdf?_gl=1*nkotui*_gcl_au*MTM1MDU3OTk5Ny4xNzg2NDU0Mzc2Li0uLS4xNzg2NDU0MzgxLjE5ODgzMTQ2NTEuMTc4NjQ1NDM4MS4xNzg2NDU0Mzgx"
+			(at 165.1 82.55 0)
+			(hide yes)
+			(show_name no)
+			(do_not_autoplace no)
+			(effects
+				(font
+					(size 1.27 1.27)
+				)
+			)
+		)
